File: Zavrsni/Zavrsni.kicad_pcb (KiCad board)
At the start: 2 copper layers, 104 x 58.3 mm, 23 parts, among them J1 12V Source, J3 Output A, J4 Pin za Vin, J5 Conn_01x04, J6 Conn_02x19_Odd_Even, J7 Conn_02x19_Odd_Even, J8 Conn_01x06, U1 LM78M05_TO220, U2 L298N

Commit message: Plot
Routing:
- net OUT2: track 24.4 -> 28.9 mm
- net 5V: track 61.5 -> 60.7 mm
Other:
- outline, holes or cut-outs redrawn
- board text added: "Zavrsni rad - Compact v1.0. Ivan Hodak"
- board text removed: "Zavrsni rad - compact v1.0. Ivan Hodak"

Commit message: Plot
Parts:
- moved Vin 4.06 mm to (212.2, 117.0)
- renumbered J4 to Vin
Routing:
- net 5V: track 60.7 -> 59.7 mm
Changed lines of the file:
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@@
 		)
 		(property "Value" "12V Source"
-			(at 1.27 4.51 0)
+			(at 1.35 5.01 0)
 			(layer "F.Fab")
 			(effects
@@
 	(footprint "Connector_PinHeader_2.54mm:PinHeader_1x01_P2.54mm_Vertical"
 		(layer "F.Cu")
-		(at 216.19 117.99)
+		(at 212.25 117)
 		(descr "Through hole straight pin header, 1x01, 2.54mm pitch, single row")
 		(tags "Through hole pin header THT 1x01 2.54mm single row")
-		(property "Reference" "J4"
-			(at 2.56 0.01 270)
+		(property "Reference" "Vin"
+			(at 0 2.75 180)
 			(layer "F.SilkS")
 			(effects
@@
 		)
 		(property "Value" "Pin za Vin"
-			(at -5.69 0.76 0)
+			(at 5.75 -0.75 0)
 			(layer "F.Fab")
 			(effects
@@
 		(tags "LED")
 		(property "Reference" "D1"
-			(at 1.27 -3.96 0)
+			(at -2.665 0.01 90)
 			(layer "F.SilkS")
 			(effects
@@
 	)
 	(segment
-		(start 210.69 133.24)
-		(end 210.69 131.24)
+		(start 210.251708 117)
+		(end 203.139 109.887292)
 		(width 0.5)
 		(layer "F.Cu")
@@
 	)
 	(segment
-		(start 196.02 98.78)
-		(end 198.21 96.59)
+		(start 210.69 133.24)
+		(end 210.69 131.24)
 		(width 0.5)
 		(layer "F.Cu")
@@
 	)
 	(segment
-		(start 197.649 100.409)
-		(end 198.732324 100.409)
+		(start 196.02 98.78)
+		(end 198.21 96.59)
 		(width 0.5)
 		(layer "F.Cu")
@@
 	)
 	(segment
-		(start 196.02 98.78)
-		(end 197.649 100.409)
+		(start 212.25 117)
+		(end 210.251708 117)
 		(width 0.5)
 		(layer "F.Cu")
@@
 	)
 	(segment
-		(start 217.015 123.19)
-		(end 216.25 122.425)
+		(start 213.5 117)
+		(end 212.25 117)
 		(width 0.5)
 		(layer "F.Cu")
@@
 	)
 	(segment
-		(start 203.139 104.815676)
-		(end 203.139 109.887292)
+		(start 197.649 100.409)
+		(end 198.732324 100.409)
 		(width 0.5)
 		(layer "F.Cu")
@@
 	)
 	(segment
-		(start 203.139 109.887292)
-		(end 211.241708 117.99)
+		(start 196.02 98.78)
+		(end 197.649 100.409)
 		(width 0.5)
 		(layer "F.Cu")
@@
 	)
 	(segment
-		(start 198.732324 100.409)
-		(end 203.139 104.815676)
+		(start 217.015 123.19)
+		(end 216.25 122.425)
 		(width 0.5)
 		(layer "F.Cu")
@@
 	)
 	(segment
-		(start 216.19 119.69)
-		(end 216.25 119.75)
+		(start 203.139 104.815676)
+		(end 203.139 109.887292)
 		(width 0.5)
 		(layer "F.Cu")
@@
 	)
 	(segment
-		(start 216.19 117.99)
-		(end 216.19 119.69)
+		(start 198.732324 100.409)
+		(end 203.139 104.815676)
 		(width 0.5)
 		(layer "F.Cu")
@@
 	)
 	(segment
-		(start 211.241708 117.99)
-		(end 216.19 117.99)
+		(start 216.25 119.75)
+		(end 213.5 117)
 		(width 0.5)
 		(layer "F.Cu")

Commit message: update
Parts:
- removed D2, D3, D6, D7: D_Schottky_Filled, Diode_THT:D_DO-41_SOD81_P12.70mm_Horizontal
- moved JP2 39.9 mm to (223.8, 125.8)
- moved D9 33.5 mm to (190.8, 106.2), turned to 90 degrees
- moved R1 32.6 mm to (191.0, 119.2)
- moved J1 23.6 mm to (208.5, 115.8), turned to 90 degrees
- moved C2 21.0 mm to (196.0, 118.3), turned to -90 degrees
- moved J5 19.6 mm to (137.2, 140.0), turned to -90 degrees
- moved D1 19.4 mm to (200.0, 125.8), turned to 180 degrees
- moved U1 17.2 mm to (201.5, 111.5), turned to 180 degrees
- moved D5 16.9 mm to (195.8, 93.5), turned to -90 degrees
- moved D8 15.5 mm to (211.0, 102.7), turned to 90 degrees
- moved C1 14.0 mm to (201.8, 118.3)
- moved J4 10.6 mm to (211.0, 106.5)
- moved JP1 10.5 mm to (209.8, 121.0), turned to -90 degrees
- moved D4 3.76 mm to (212.3, 84.8), turned to 180 degrees
- moved U2 3.75 mm to (198.9, 90.1)
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- renumbered Vin to J4
Connections:
- U2 pad 13: Net-(D3-K) -> unconnected-(U2-OUT3-Pad13)
- U2 pad 14: Net-(D2-K) -> unconnected-(U2-OUT4-Pad14)
Routing:
- net 12V: track 87.3 -> 0.00 mm
- net 5V BL: track 70.6 -> 0.00 mm
- net 5V: track 59.7 -> 0.00 mm, vias 2 -> 0
- net 3V3: track 52.2 -> 0.00 mm
- net SCL: track 47.1 -> 0.00 mm
- net SDA: track 43.9 -> 0.00 mm
- net RX: track 31.7 -> 0.00 mm
- net OUT2: track 28.9 -> 0.00 mm
- net OUT1: track 24.7 -> 0.00 mm, vias 2 -> 0
- net Net-(D3-K): track 21.2 -> 0.00 mm, vias 2 -> 0
- net TX: track 15.4 -> 0.00 mm
- net IN1: track 13.5 -> 0.00 mm
- net IN2: track 13.5 -> 0.00 mm
- net Net-(D2-K): track 11.7 -> 0.00 mm
- net Net-(JP2-B): track 10.4 -> 0.00 mm
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Other:
- board size 104 x 58.3 mm -> 94.2 x 61.2 mm

Commit message: New
Parts:
- removed JP2: Jumper_Bridged, Connector_PinHeader_2.54mm:PinHeader_1x02_P2.54mm_Vertical
- moved J8 12.9 mm to (172.9, 140.8), turned to 90 degrees
- moved JP1 8.25 mm to (210.0, 112.8)
- moved C1 6.05 mm to (203.5, 112.5), turned to 180 degrees
- moved C2 5.82 mm to (196.5, 112.5), turned to 180 degrees
- moved U1 5.55 mm to (201.5, 117.0)
- moved J1 4.32 mm to (209.2, 120.0)
- moved D1 3.91 mm to (197.0, 123.2), turned to -90 degrees
- moved R1 0.86 mm to (191.5, 118.5)
- moved J5 0.78 mm to (137.2, 140.8)
- moved J3 0.56 mm to (195.0, 86.5)
Connections:
- J6 pad 17: 5V BL -> unconnected-(J6-Pin_17-Pad17)
- J6 pad 5: unconnected-(J6-Pin_5-Pad5) -> 5V
- J8 pad 2: 5V BL -> 5V
- U2 pad 6: Net-(JP2-B) -> 5V
Routing:
- net 5V: track 0.00 -> 171.9 mm
- net SCL: track 0.00 -> 63.4 mm
- net 12V: track 0.00 -> 50.2 mm
- net SDA: track 0.00 -> 43.9 mm
- net 3V3: track 0.00 -> 41.0 mm
- net RX: track 0.00 -> 31.5 mm
- net OUT1: track 0.00 -> 24.4 mm
- net IN1: track 0.00 -> 21.0 mm
- net IN2: track 0.00 -> 20.1 mm
- net TX: track 0.00 -> 16.3 mm
- net OUT2: track 0.00 -> 16.3 mm
- net Net-(D1-A): track 0.00 -> 8.77 mm
- net Net-(JP1-B): track 0.00 -> 7.74 mm
Other:
- board text added: "Zavrsni rad - Compact v1.1. Ivan Hodak"
- board text removed: "Zavrsni rad - Compact v1.0. Ivan Hodak"

Commit message: New
Parts:
- removed J4: Pin za Vin, Connector_PinHeader_2.54mm:PinHeader_1x01_P2.54mm_Vertical
- added H1: MountingHole, MountingHole:MountingHole_2.2mm_M2_ISO7380, F.Cu at (113.9, 79.2)
- added H2: MountingHole, MountingHole:MountingHole_2.2mm_M2_ISO7380, F.Cu at (211.2, 79.2)
- added H3: MountingHole, MountingHole:MountingHole_2.2mm_M2_ISO7380, F.Cu at (113.9, 134.5)
- added H4: MountingHole, MountingHole:MountingHole_2.2mm_M2_ISO7380, F.Cu at (211.2, 134.5)
- moved J5 37.7 mm to (114.8, 110.5), turned to 180 degrees
- moved J8 21.5 mm to (191.9, 130.8)
Connections:
- C2 pad 1: 5V -> Vss
- J6 pad 17: unconnected-(J6-Pin_17-Pad17) -> 5V
- J6 pad 23: unconnected-(J6-Pin_23-Pad23) -> 12V
- J6 pad 5: 5V -> unconnected-(J6-Pin_5-Pad5)
- R1 pad 1: 5V -> Vss
- U1 pad 3: 5V -> Vss
- U2 pad 6: 5V -> Vss
- U2 pad 9: 5V -> Vss
Routing:
- net 5V: track 171.9 -> 86.4 mm
- net 12V: track 50.2 -> 119.1 mm
- net SDA: track 43.9 -> 7.98 mm
- net Vss: track 0.00 -> 30.2 mm, vias 0 -> 2
- net 3V3: track 41.0 -> 11.2 mm
- net SCL: track 63.4 -> 71.3 mm
- net TX: track 16.3 -> 18.2 mm
- net RX: track 31.5 -> 30.2 mm
Other:
- board size 94.2 x 61.2 mm -> 103.4 x 61.2 mm
- board text added: "Zavrsni rad - Compact v1.2 Ivan Hodak"
- board text removed: "Zavrsni rad - Compact v1.1. Ivan Hodak"

Commit message: New
Parts:
- moved C1 11.0 mm to (193.2, 108.5), turned to -90 degrees
- moved H3 4.00 mm to (113.8, 130.5)
- moved H4 4.00 mm to (211.2, 130.5)
- moved D5 3.50 mm to (195.8, 90.0)
- moved D9 3.50 mm to (190.8, 102.7)
- moved C2 2.50 mm to (199.0, 112.5), turned to 0 degrees
- moved H1 1.75 mm to (113.8, 81.0)
- moved H2 1.75 mm to (211.2, 81.0)
- moved J3 1.75 mm to (195.0, 84.8)
- moved D4 1.25 mm to (211.3, 85.5)
- moved J8 0.50 mm to (191.9, 130.2)
Routing:
- net 12V: track 119.1 -> 122.6 mm
- net IN2: track 20.1 -> 17.7 mm
- net IN1: track 21.0 -> 18.6 mm
- net Vss: track 30.2 -> 31.4 mm
- net OUT2: track 16.3 -> 15.2 mm
- net 5V: track 86.4 -> 87.2 mm
- net RX: track 30.2 -> 29.7 mm
Other:
- board size 103.4 x 61.2 mm -> 103.5 x 55.5 mm
- board text added: "Zavrsni rad Ivan Hodak, 2026."
- board text removed: "Zavrsni rad - Compact v1.2 Ivan Hodak"

Commit message: New 3
Parts:
- moved D1 7.27 mm to (196.5, 130.5), turned to 90 degrees
- moved J8 6.99 mm to (195.0, 124.0)
- moved H1 1.68 mm to (115.2, 81.8)
- moved H3 1.52 mm to (115.2, 130.2)
- moved H2 0.90 mm to (210.8, 81.8)
- moved H4 0.71 mm to (210.8, 130.0)
- moved J5 0.50 mm to (115.2, 110.5)
- moved J1 0.35 mm to (209.0, 119.8)
Routing:
- net TX: track 18.0 -> 22.8 mm
- net Net-(D1-A): track 8.77 -> 9.98 mm
- net 5V: track 87.2 -> 88.4 mm
- net SCL: track 71.3 -> 70.3 mm
Other:
- board size 103.5 x 55.5 mm -> 100.9 x 53.5 mm

Commit message: New 4
Parts:
- H1, H2, H3, H4: footprint MountingHole:MountingHole_2.2mm_M2_ISO7380 -> MountingHole:MountingHole_3mm
- R1: footprint Resistor_SMD:R_1206_3216Metric_Pad1.30x1.75mm_HandSolder -> Resistor_THT:R_Axial_DIN0204_L3.6mm_D1.6mm_P5.08mm_Horizontal
- moved D1 19.8 mm to (196.4, 110.7), turned to -90 degrees
- moved C2 14.9 mm to (209.7, 122.8), turned to 90 degrees
- moved D8 12.7 mm to (199.1, 107.1)
- moved C1 11.1 mm to (202.6, 114.5)
- moved JP1 9.83 mm to (203.7, 120.3)
- moved U1 7.39 mm to (204.0, 124.0)
- moved R1 7.13 mm to (198.0, 121.4), turned to 90 degrees
- moved J8 6.34 mm to (194.3, 117.7), turned to 0 degrees
- moved U2 4.40 mm to (202.3, 92.9)
- moved D4 4.00 mm to (211.3, 89.5)
- moved J1 2.88 mm to (209.4, 116.9)
- moved H2 2.56 mm to (210.0, 84.2)
- moved H1 2.53 mm to (115.9, 84.2)
- moved D5 2.23 mm to (195.0, 92.1)
- moved J3 2.17 mm to (194.7, 86.9)
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Routing:
- net Vss: track 31.4 -> 56.9 mm, vias 2 -> 0
- net 5V: track 88.4 -> 77.4 mm
- net TX: track 22.8 -> 12.0 mm
- net IN1: track 18.6 -> 28.0 mm
- net IN2: track 17.7 -> 26.6 mm
- net Net-(D1-A): track 9.98 -> 3.76 mm
- net RX: track 29.9 -> 24.9 mm
- net OUT2: track 15.2 -> 19.2 mm
- net Net-(JP1-B): track 7.74 -> 4.88 mm
- net 12V: track 122.7 -> 120.5 mm, vias 0 -> 1
- net OUT1: track 24.0 -> 25.7 mm
Other:
- board size 100.9 x 53.5 mm -> 100.9 x 51.9 mm
