File: Zavrsni/Zavrsni.kicad_pcb (KiCad board)
At the start: 2 copper layers, 100.9 x 51.9 mm, 21 parts, among them J1 12V Source, J3 Output A, J5 Conn_01x04, J6 Conn_02x19_Odd_Even, J7 Conn_02x19_Odd_Even, J8 Conn_01x06, U1 LM78M05_TO220, U2 L298N

Commit message: Final
Parts:
- removed JP1: Jumper_Bridged, Connector_PinHeader_2.54mm:PinHeader_1x02_P2.54mm_Vertical
- moved U1 3.53 mm to (201.7, 121.4), turned to -90 degrees
Connections:
- U1 pad 1: Net-(JP1-B) -> 12V
Routing:
- net Net-(JP1-B): track 4.88 -> 0.00 mm
- net 12V: track 120.5 -> 121.3 mm
- net Vss: track 56.9 -> 57.5 mm
