File: Zavrsni/Zavrsni.kicad_sch (KiCad schematic)
At the start: 19 parts, among them J1 12V Source, J2 Input, J3 Output A, U1 LM78M05_TO220, U2 L298N

Commit message: upd
Parts:
- added J4: Pin za Vin, Connector_PinHeader_2.54mm:PinHeader_1x01_P2.54mm_Vertical, symbol Connector:Conn_01x01_Pin
- added J6, J7: Conn_02x19_Odd_Even, Connector_PinSocket_2.54mm:PinSocket_2x19_P2.54mm_Vertical, symbol Connector_Generic:Conn_02x19_Odd_Even
Connections:
- net 12V: now also D6.1 (K), D7.1 (K), D8.1 (K), D9.1 (K)
- net 5V: now also J4.1 (Pin_1)
- net GND: now also D2.2 (A), D3.2 (A), D4.2 (A), D5.2 (A), U2.1 (SENSE_A), U2.15 (SENSE_B), U2.8 (GND)
- net OUT1: now reaches D4.1 (K)
- net OUT1: now also D8.2 (A), J3.1 (Pin_1), U2.2 (OUT1)
- net at U2.13 (OUT3): now also D3.1 (K), D7.2 (A)
- net at U2.14 (OUT4): now also D2.1 (K), D6.2 (A)
- net OUT2: now reaches U2.3 (OUT2)
- net OUT2: now also D5.1 (K), D9.2 (A), J3.2 (Pin_2)
- no-connect marks 0 -> 70
Other:
- note added: "Od jedne do druge strane nasuprotnih socketa ima 63.5mm"
- moved on the sheet: C1, C2, D1, D2, D3, D4, D5, D6, D7, D8, D9, J1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

Commit message: Big Update
Parts:
- removed J2: Input, symbol Connector:Screw_Terminal_01x02
- added J5: Conn_01x04, Connector_PinSocket_2.54mm:PinSocket_1x04_P2.54mm_Vertical, symbol Connector_Generic:Conn_01x04
- added J8: Conn_01x06, Connector_PinSocket_2.54mm:PinSocket_1x06_P2.54mm_Vertical, symbol Connector_Generic:Conn_01x06
- C1, C2: footprint (none) -> Capacitor_THT:CP_Radial_D5.0mm_P2.00mm
- D1: footprint (none) -> LED_THT:LED_D5.0mm
- D2, D3, D4, D5, D6, D7, D8, D9: footprint (none) -> Diode_THT:D_DO-41_SOD81_P12.70mm_Horizontal
- J1, J3: footprint (none) -> TerminalBlock_Phoenix:TerminalBlock_Phoenix_MPT-0,5-2-2.54_1x02_P2.54mm_Horizontal
- JP1, JP2: footprint (none) -> Connector_PinHeader_2.54mm:PinHeader_1x02_P2.54mm_Vertical
- R1: footprint (none) -> Resistor_SMD:R_1206_3216Metric_Pad1.30x1.75mm_HandSolder
- U2: footprint Package_TO_SOT_THT:TO-220-15_P2.54x5.08mm_StaggerOdd_Lead4.58mm_Vertical -> L298N:TO127P2020X500X2100-15
Connections:
- net GND: now also J6.19 (Pin_19), J5.3 (Pin_3), J8.3 (Pin_3)
- net IN1: now reaches U2.5 (IN1)
- net IN1: now also J7.1 (Pin_1)
- net IN2: now reaches U2.7 (IN2)
- net IN2: now also J7.3 (Pin_3)
- net SCL: now reaches J7.18 (Pin_18)
- net SCL: now also J5.2 (Pin_2)
- net RX: now reaches J7.22 (Pin_22)
- net RX: now also J8.5 (Pin_5)
- net TX: now reaches J7.34 (Pin_34)
- net TX: now also J8.4 (Pin_4)
- net GUMB: now reaches J7.5 (Pin_5)
- net 3V3: now reaches J6.15 (Pin_15)
- net 3V3: now also J5.4 (Pin_4)
- net 5V BL: now reaches J6.17 (Pin_17)
- net 5V BL: now also J8.2 (Pin_2)
- net SDA: now reaches J6.22 (Pin_22)
- net SDA: now also J5.1 (Pin_1)
- no-connect marks 70 -> 71
Other:
- note added: "Socketi za senzor i bluetooth"
- moved on the sheet: C1, C2, D1, D2, D3, D4, D5, D6, D7, D8, D9, J1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

Commit message: Plot
Parts:
- U2: Manufacturer (none) -> STMicroelectronics; Manufacturer part number (none) -> L298
Changed lines of the file:
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@@
+			)
+		)
+		(property "Manufacturer" "STMicroelectronics"
+			(at 88.9 96.52 0)
+			(effects
+				(font
+					(size 1.27 1.27)
+				)
+				(hide yes)
+			)
+		)
+		(property "Manufacturer part number" "L298"
+			(at 88.9 96.52 0)
+			(effects
+				(font
+					(size 1.27 1.27)
+				)
+				(hide yes)
 			)
 		)
@@
 			)
 		)
+		(property "Manufacturer" ""
+			(at 118.11 45.72 90)
+			(effects
+				(font
+					(size 1.27 1.27)
+				)
+				(hide yes)
+			)
+		)
+		(property "Manufacturer part number" ""
+			(at 118.11 45.72 90)
+			(effects
+				(font
+					(size 1.27 1.27)
+				)
+				(hide yes)
+			)
+		)
 		(pin "2"
 		)
@@
 			)
 		)
+		(property "Manufacturer" ""
+			(at 90.17 29.21 0)
+			(effects
+				(font
+					(size 1.27 1.27)
+				)
+				(hide yes)
+			)
+		)
+		(property "Manufacturer part number" ""
+			(at 90.17 29.21 0)
+			(effects
+				(font
+					(size 1.27 1.27)
+				)
+				(hide yes)
+			)
+		)
 		(pin "2"
 		)
@@
 			)
 		)
+		(property "Manufacturer" ""
+			(at 104.14 35.56 0)
+			(effects
+				(font
+					(size 1.27 1.27)
+				)
+				(hide yes)
+			)
+		)
+		(property "Manufacturer part number" ""
+			(at 104.14 35.56 0)
+			(effects
+				(font
+					(size 1.27 1.27)
+				)
+				(hide yes)
+			)
+		)
 		(pin "1"
 		)
@@
 			)
 		)
+		(property "Manufacturer" ""
+			(at 64.77 35.56 0)
+			(effects
+				(font
+					(size 1.27 1.27)
+				)
+				(hide yes)
+			)
+		)
+		(property "Manufacturer part number" ""
+			(at 64.77 35.56 0)
+			(effects
+				(font
+					(size 1.27 1.27)
+				)
+				(hide yes)
+			)
+		)
 		(pin "1"
 		)
@@
 			(at 118.11 35.56 0)
 			(effects
+				(font
+					(size 1.27 1.27)
+				)
+				(hide yes)
+			)
+		)
+		(property "Manufacturer" ""
+			(at 118.11 35.56 0)
+			(effects
+				(font
+					(size 1.27 1.27)
+				)
+				(hide yes)
+			)
+		)
+		(property "Manufacturer part number" ""
+			(at 118.11 35.56 0)
+			(effects

Commit message: update
Parts:
- removed D2, D3, D6, D7: D_Schottky_Filled, Diode_THT:D_DO-41_SOD81_P12.70mm_Horizontal, symbol Device:D_Schottky_Filled
- removed JP2: Jumper_Bridged, Connector_PinHeader_2.54mm:PinHeader_1x02_P2.54mm_Vertical, symbol Jumper:Jumper_2_Bridged
Connections:
- net 5V: now also U2.6 (EnA)
- no-connect marks 71 -> 73
Other:
- moved on the sheet: D4, D5, D8, D9

Commit message: New
Parts:
- removed J4: Pin za Vin, Connector_PinHeader_2.54mm:PinHeader_1x01_P2.54mm_Vertical, symbol Connector:Conn_01x01_Pin
- U1: Manufacturer (none) -> ONSEMI; Manufacturer part number (none) -> TO-220
Connections:
- net 5V: now also J6.5 (Pin_5), J8.2 (Pin_2)
- net 5V BL: no longer names the net of J6.17 (Pin_17)
- net 5V BL: no longer J8.2 (Pin_2)
Other:
- note added: "LM78M05 i L298N"
- note added: "Socketi za STM"

Commit message: New
Parts:
- added H1, H2, H3, H4: MountingHole, MountingHole:MountingHole_2.2mm_M2_ISO7380, symbol Mechanical:MountingHole
Connections:
- net 12V: now also J6.23 (Pin_23)
- net 5V: now also J6.17 (Pin_17); no longer C2.1, J6.5 (Pin_5), R1.1, U1.3 (VO), U2.6 (EnA), U2.9 (Vss)
- new net Vss: C2.1, R1.1, U1.3 (VO), U2.6 (EnA), U2.9 (Vss)
- no-connect marks 73 -> 72
Other:
- note added: "HC-05 socketi"
- note added: "L298N"
- note added: "LM78M05"
- note added: "SHT21 socketi"
- note removed: "LM78M05 i L298N"
- note removed: "Socketi za senzor i bluetooth"
- company: (none) -> TVZ
- title: (none) -> Zavrsni rad
- moved on the sheet: C1, C2, D1, D4, D5, D8, D9, J1, J3, J6, J7, JP1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

Commit message: New 4
Parts:
- H1, H2, H3, H4: footprint MountingHole:MountingHole_2.2mm_M2_ISO7380 -> MountingHole:MountingHole_3mm
- R1: footprint Resistor_SMD:R_1206_3216Metric_Pad1.30x1.75mm_HandSolder -> Resistor_THT:R_Axial_DIN0204_L3.6mm_D1.6mm_P5.08mm_Horizontal
Changed lines of the file:
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@@
 			)
 		)
-		(property "Footprint" "MountingHole:MountingHole_2.2mm_M2_ISO7380"
+		(property "Footprint" "MountingHole:MountingHole_3mm"
 			(at 158.75 190.5 0)
 			(effects
@@
 			)
 		)
-		(property "Footprint" "MountingHole:MountingHole_2.2mm_M2_ISO7380"
+		(property "Footprint" "MountingHole:MountingHole_3mm"
 			(at 158.75 171.45 0)
 			(effects
@@
 			)
 		)
-		(property "Footprint" "MountingHole:MountingHole_2.2mm_M2_ISO7380"
+		(property "Footprint" "MountingHole:MountingHole_3mm"
 			(at 158.75 177.8 0)
 			(effects
@@
 			)
 		)
-		(property "Footprint" "MountingHole:MountingHole_2.2mm_M2_ISO7380"
+		(property "Footprint" "MountingHole:MountingHole_3mm"
 			(at 158.75 184.15 0)
 			(effects
@@
 			)
 		)
-		(property "Footprint" "Resistor_SMD:R_1206_3216Metric_Pad1.30x1.75mm_HandSolder"
+		(property "Footprint" "Resistor_THT:R_Axial_DIN0204_L3.6mm_D1.6mm_P5.08mm_Horizontal"
 			(at 126.492 41.91 90)
 			(effects

Commit message: Final
Parts:
- removed JP1: Jumper_Bridged, Connector_PinHeader_2.54mm:PinHeader_1x02_P2.54mm_Vertical, symbol Jumper:Jumper_2_Bridged
Connections:
- net 12V: now also U1.1 (VI)
Changed lines of the file:
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@@
 	(wire
 		(pts
-			(xy 74.93 35.56) (xy 80.01 35.56)
+			(xy 74.93 35.56) (xy 92.71 35.56)
 		)
 		(stroke
@@
 		(pts
 			(xy 82.55 148.59) (xy 82.55 151.13)
-		)
-		(stroke
-			(width 0)
-			(type default)
-		)
-	)
-	(wire
-		(pts
-			(xy 90.17 35.56) (xy 92.71 35.56)
 		)
 		(stroke
@@
 					(unit 1)
 				)
-			)
-		)
-	)
-	(symbol
-		(lib_id "Jumper:Jumper_2_Bridged")
-		(at 85.09 35.56 0)
-		(unit 1)
-		(exclude_from_sim no)
-		(in_bom yes)
-		(on_board yes)
-		(dnp no)
-		(fields_autoplaced yes)
-		(property "Reference" "JP1"
-			(at 85.09 30.48 0)
-			(effects
-				(font
-					(size 1.27 1.27)
-				)
-			)
-		)
-		(property "Value" "Jumper_Bridged"
-			(at 85.09 33.02 0)
-			(effects
-				(font
-					(size 1.27 1.27)
-				)
-			)
-		)
-		(property "Footprint" "Connector_PinHeader_2.54mm:PinHeader_1x02_P2.54mm_Vertical"
-			(at 85.09 35.56 0)
-			(effects
-				(font
-					(size 1.27 1.27)
-				)
-				(hide yes)
-			)
-		)
-		(property "Datasheet" "~"
-			(at 85.09 35.56 0)
-			(effects
-				(font
-					(size 1.27 1.27)
-				)
-				(hide yes)
-			)
-		)
-		(property "Description" "Jumper, 2-pole, closed/bridged"
-			(at 85.09 35.56 0)
-			(effects
-				(font
-					(size 1.27 1.27)
-				)
-				(hide yes)
-			)
-		)
-		(pin "1"
-		)
-		(pin "2"
-		)
-		(instances
-			(project ""
-				(path "/f2ac0668-a3c8-4093-af03-acd91b31ec7e"
-					(reference "JP1")
-					(unit 1)
-				)
